File: Rev. A/ZX81 Composite.kicad_pcb (KiCad board)
At the start: 2 copper layers, 37.1 x 24.1 mm, 16 parts, among them J1 +5 Volt Input, J2 ULA Pin 16, J3 Video Out, Q1 BC337, Q2 BC337, U1 NE555

Commit message: Add files via upload
Connections:
- R3 pad 1: Net-(Q1-Pad3) -> Net-(D1-Pad2)
Routing:
- net Net-(D1-Pad2): track 14.5 -> 20.2 mm
- net Net-(Q1-Pad3): track 33.8 -> 29.6 mm
