File: Rev. A/ZX81 Composite.sch (KiCad schematic (older format))
At the start: 16 parts, among them J1 +5 Volt Input, J2 ULA Pin 16, J3 Video Out, Q1 BC337, Q2 BC337, U1 NE555

Commit message: Add files via upload
Connections:
- net at Q1.3 (E), R4.1: no longer R3.1
- net at D1.2 (A), R4.2: now also R3.1
Changed lines of the file:
@@
 	6700 1950 6700 2300
-$Comp
-L Device:R R4
-U 1 1 60640DC9
-P 6700 3250
-F 0 "R4" H 6770 3296 50  0000 L CNN
-F 1 "56R" H 6770 3205 50  0000 L CNN
-F 2 "Resistors_THT:R_Axial_DIN0204_L3.6mm_D1.6mm_P5.08mm_Horizontal" V 6630 3250 50  0001 C CNN
-F 3 "~" H 6700 3250 50  0001 C CNN
-	1    6700 3250
-	1    0    0    -1
-$EndComp
 $Comp
 L ZX81-Composite-rescue:NE555-Timer U1
@@
 $EndComp
 Wire Wire Line
-	6700 3400 6700 3600
-Wire Wire Line
 	5300 3250 5450 3250
 Connection ~ 5300 3250
@@
 	1    0    0    -1
 $EndComp
-Wire Wire Line
-	6700 2700 6700 3050
 $Comp
 L Device:R R3
@@
 Wire Wire Line
 	6650 3050 6700 3050
-Connection ~ 6700 3050
-Wire Wire Line
-	6700 3050 6700 3100
 Wire Wire Line
 	6300 3450 6300 5200
@@
 Text Label 3050 1950 0    50   ~ 0
 +5V
+$Comp
+L Device:R R4
+U 1 1 60A688D3
+P 6700 2850
+F 0 "R4" H 6770 2896 50  0000 L CNN
+F 1 "56R" H 6770 2805 50  0000 L CNN
+F 2 "Resistors_THT:R_Axial_DIN0204_L3.6mm_D1.6mm_P5.08mm_Horizontal" V 6630 2850 50  0001 C CNN
+F 3 "~" H 6700 2850 50  0001 C CNN
+	1    6700 2850
+	1    0    0    -1
+$EndComp
+Wire Wire Line
+	6700 3000 6700 3050
+Connection ~ 6700 3050
+Wire Wire Line
+	6700 3050 6700 3600
 $EndSCHEMATC
